File: hardware/pcb/v1/rpi-pico-sao-host.kicad_pcb (KiCad board)
At the start: 2 copper layers, 42 x 51.5 mm, 11 parts, among them J1 SAO Host Header, J2 SAO Host Header

Commit message: WIP
Parts:
- A1: value RaspberryPi Pico W -> Raspberry Pi Pico; footprint rpi-pico-sao-host:RASPBERRY_PI_PICO_W -> rpi-pico-sao-host:RASPBERRY_PI_PICO_COMMON_MOUNTINGHOLES
