File: hardware/pcb/v1/rpi-pico-sao-host.kicad_sch (KiCad schematic)
At the start: 12 parts, among them J1 SAO Host Header, J2 SAO Host Header

Commit message: WIP
Parts:
- A1: value RaspberryPi Pico W -> Raspberry Pi Pico; footprint rpi-pico-sao-host:RASPBERRY_PI_PICO_W -> rpi-pico-sao-host:RASPBERRY_PI_PICO_COMMON_MOUNTINGHOLES; symbol rpi-pico-sao-host:PCA_RaspberryPi_Pico_W -> rpi-pico-sao-host:PCA_Raspberry_Pi_Pico; Manufacturer Part Number SC0918 -> SC0915
Connections:
- net GND: no longer A1.D2 (GND)
- no-connect marks 31 -> 24
Changed lines of the file:
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@@
-	)
-	(no_connect
-		(at 71.12 60.96)
-	)
-	(no_connect
-		(at 116.84 68.58)
-	)
-	(no_connect
-		(at 116.84 63.5)
-	)
-	(no_connect
-		(at 71.12 58.42)
-	)
-	(no_connect
-		(at 71.12 116.84)
 	)
 	(no_connect
@@
 	)
 	(no_connect
-		(at 116.84 60.96)
-	)
-	(no_connect
 		(at 71.12 91.44)
 	)
@@
 	(no_connect
 		(at 116.84 88.9)
-	)
-	(no_connect
-		(at 116.84 58.42)
 	)
 	(wire
@@
 	)
 	(symbol
-		(lib_id "rpi-pico-sao-host:PCA_RaspberryPi_Pico_W")
+		(lib_id "rpi-pico-sao-host:PCA_Raspberry_Pi_Pico")
 		(at 93.98 88.9 0)
 		(unit 1)
@@
 			)
 		)
-		(property "Value" "RaspberryPi Pico W"
+		(property "Value" "Raspberry Pi Pico"
 			(at 101.6 50.8 0)
 			(effects
@@
 			)
 		)
-		(property "Footprint" "rpi-pico-sao-host:RASPBERRY_PI_PICO_W"
+		(property "Footprint" "rpi-pico-sao-host:RASPBERRY_PI_PICO_COMMON_MOUNTINGHOLES"
+			(at 93.98 148.59 0)
+			(effects
+				(font
+					(size 1.27 1.27)
+				)
+				(hide yes)
+			)
+		)
+		(property "Datasheet" "https://datasheets.raspberrypi.com/pico/pico-datasheet.pdf"
+			(at 93.98 146.05 0)
+			(effects
+				(font
+					(size 1.27 1.27)
+				)
+				(hide yes)
+			)
+		)
+		(property "Description" "Versatile and inexpensive microcontroller module powered by RP2040 dual-core Arm Cortex-M0+ processor up to 133 MHz, 264kB SRAM, 2MB QSPI flash"
+			(at 93.98 143.51 0)
+			(effects
+				(font
+					(size 1.27 1.27)
+				)
+				(hide yes)
+			)
+		)
+		(property "Manufacturer" "Raspberry Pi"
 			(at 93.98 138.43 0)
 			(effects
@@
 			)
 		)
-		(property "Datasheet" "https://datasheets.raspberrypi.com/picow/pico-w-datasheet.pdf"
+		(property "Manufacturer Part Number" "SC0915"
 			(at 93.98 140.97 0)
 			(effects
@@
 			)
 		)
-		(property "Description" "RASPBERRY PI PICO W RP2040"
-			(at 93.98 143.51 0)
-			(effects
-				(font
-					(size 1.27 1.27)
-				)
-				(hide yes)
-			)
-		)
-		(property "Manufacturer" "Raspberry Pi"
-			(at 95.25 146.05 0)
-			(effects
-				(font
-					(size 1.27 1.27)
-				)
-				(hide yes)
-			)
-		)
-		(property "Manufacturer Part Number" "SC0918"
-			(at 93.98 148.59 0)
-			(effects
-				(font
-					(size 1.27 1.27)
-				)
-				(hide yes)
-			)
-		)
 		(pin "10"
 		)
@@
 		(pin "9"
 		)
-		(pin "D1"
-		)
-		(pin "D2"
-		)
-		(pin "D3"
-		)
-		(pin "TP1"
-		)
-		(pin "TP2"
-		)
-		(pin "TP3"
-		)
-		(pin "TP4"
-		)
-		(pin "TP5"
-		)
-		(pin "TP6"
-		)
 		(instances
